Commit message: Decreased alpha values of robots's base link, changed the wheels' rotation axis from y to z.

File: my_rb1_description/urdf/my_rb1_robot.urdf (robot description, URDF)
Before this commit: robot my_rb1_robot, 7 links, 6 joints
Joints:
- joint left_wheel_joint: axis 0 1 0 -> 0 0 1
- joint right_wheel_joint: axis 0 1 0 -> 0 0 1
